Commit message: Refactor: name description

File: urdf/IRRobot_description/urdf/IRRobot.xacro (robot description, xacro)
@@ -1,7 +1,7 @@
 <?xml version="1.0" ?>
-<robot name="IRRobot" xmlns:xacro="http://www.ros.org/wiki/xacro">
-<xacro:include filename="$(find IRRobot_description)/urdf/materials.xacro" />
-<xacro:include filename="$(find IRRobot_description)/urdf/IRRobot.trans" />
-<xacro:include filename="$(find IRRobot_description)/urdf/IRRobot.gazebo" />
+<robot name="irrobot" xmlns:xacro="http://www.ros.org/wiki/xacro">
+<xacro:include filename="$(find irrobot_description)/urdf/materials.xacro" />
+<xacro:include filename="$(find irrobot_description)/urdf/irrobot.trans" />
+<xacro:include filename="$(find irrobot_description)/urdf/irrobot.gazebo" />
 <link name="base_link">
   <inertial>
@@ -13,5 +13,5 @@
     <origin xyz="0 0 0" rpy="0 0 0"/>
     <geometry>
-      <mesh filename="file://$(find IRRobot_description)/meshes/base_link.stl" scale="0.001 0.001 0.001"/>
+      <mesh filename="file://$(find irrobot_description)/meshes/base_link.stl" scale="0.001 0.001 0.001"/>
     </geometry>
     <material name="silver"/>
@@ -20,5 +20,5 @@
     <origin xyz="0 0 0" rpy="0 0 0"/>
     <geometry>
-      <mesh filename="file://$(find IRRobot_description)/meshes/base_link.stl" scale="0.001 0.001 0.001"/>
+      <mesh filename="file://$(find irrobot_description)/meshes/base_link.stl" scale="0.001 0.001 0.001"/>
     </geometry>
   </collision>
@@ -26,5 +26,5 @@
 <link name="box_motor_1_1">
   <inertial>
-    <origin xyz="-0.010634642706834604 -0.01075607322190826 -0.013698698265978582" rpy="0 0 0"/>
+    <origin xyz="-0.010634642706834604 -0.010756073221908219 -0.013698698265978554" rpy="0 0 0"/>
     <mass value="0.0969363525800495"/>
     <inertia ixx="2.1e-05" iyy="4.3e-05" izz="3.7e-05" ixy="1e-06" iyz="-3e-06" ixz="2e-06"/>
@@ -33,5 +33,5 @@
     <origin xyz="-0.085 0.07 0.002768" rpy="0 0 0"/>
     <geometry>
-      <mesh filename="file://$(find IRRobot_description)/meshes/box_motor_1_1.stl" scale="0.001 0.001 0.001"/>
+      <mesh filename="file://$(find irrobot_description)/meshes/box_motor_1_1.stl" scale="0.001 0.001 0.001"/>
     </geometry>
     <material name="silver"/>
@@ -40,5 +40,5 @@
     <origin xyz="-0.085 0.07 0.002768" rpy="0 0 0"/>
     <geometry>
-      <mesh filename="file://$(find IRRobot_description)/meshes/box_motor_1_1.stl" scale="0.001 0.001 0.001"/>
+      <mesh filename="file://$(find irrobot_description)/meshes/box_motor_1_1.stl" scale="0.001 0.001 0.001"/>
     </geometry>
   </collision>
@@ -46,12 +46,12 @@
 <link name="box_motor_2_1">
   <inertial>
-    <origin xyz="-0.010634642706834604 0.023000000000000007 -0.013698698265978578" rpy="0 0 0"/>
+    <origin xyz="-0.010634642706834563 0.02299999999999995 -0.013698698265978537" rpy="0 0 0"/>
     <mass value="0.19387270516009888"/>
-    <inertia ixx="7.1e-05" iyy="8.6e-05" izz="0.000103" ixy="0.0" iyz="-0.0" ixz="4e-06"/>
+    <inertia ixx="7.1e-05" iyy="8.6e-05" izz="0.000103" ixy="0.0" iyz="0.0" ixz="4e-06"/>
   </inertial>
   <visual>
     <origin xyz="-0.085 -0.07 0.002768" rpy="0 0 0"/>
     <geometry>
-      <mesh filename="file://$(find IRRobot_description)/meshes/box_motor_2_1.stl" scale="0.001 0.001 0.001"/>
+      <mesh filename="file://$(find irrobot_description)/meshes/box_motor_2_1.stl" scale="0.001 0.001 0.001"/>
     </geometry>
     <material name="silver"/>
@@ -60,5 +60,5 @@
     <origin xyz="-0.085 -0.07 0.002768" rpy="0 0 0"/>
     <geometry>
-      <mesh filename="file://$(find IRRobot_description)/meshes/box_motor_2_1.stl" scale="0.001 0.001 0.001"/>
+      <mesh filename="file://$(find irrobot_description)/meshes/box_motor_2_1.stl" scale="0.001 0.001 0.001"/>
     </geometry>
   </collision>
@@ -66,12 +66,12 @@
 <link name="box_motor_3_1">
   <inertial>
-    <origin xyz="0.041600000342726734 -0.01075607322190833 -0.013698698265978585" rpy="0 0 0"/>
+    <origin xyz="0.04160000034272672 -0.010756073221908302 -0.01369869826597855" rpy="0 0 0"/>
     <mass value="0.19387270516009908"/>
-    <inertia ixx="4.2e-05" iyy="0.000272" izz="0.00026" ixy="-0.0" iyz="-6e-06" ixz="0.0"/>
+    <inertia ixx="4.2e-05" iyy="0.000272" izz="0.00026" ixy="0.0" iyz="-6e-06" ixz="0.0"/>
   </inertial>
   <visual>
     <origin xyz="0.075 0.07 0.002768" rpy="0 0 0"/>
     <geometry>
-      <mesh filename="file://$(find IRRobot_description)/meshes/box_motor_3_1.stl" scale="0.001 0.001 0.001"/>
+      <mesh filename="file://$(find irrobot_description)/meshes/box_motor_3_1.stl" scale="0.001 0.001 0.001"/>
     </geometry>
     <material name="silver"/>
@@ -80,5 +80,5 @@
     <origin xyz="0.075 0.07 0.002768" rpy="0 0 0"/>
     <geometry>
-      <mesh filename="file://$(find IRRobot_description)/meshes/box_motor_3_1.stl" scale="0.001 0.001 0.001"/>
+      <mesh filename="file://$(find irrobot_description)/meshes/box_motor_3_1.stl" scale="0.001 0.001 0.001"/>
     </geometry>
   </collision>
@@ -86,5 +86,5 @@
 <link name="box_motor_4_1">
   <inertial>
-    <origin xyz="0.051921786221357444 0.018918691073969415 -0.013698698265978592" rpy="0 0 0"/>
+    <origin xyz="0.051921786221357416 0.018918691073969318 -0.013698698265978533" rpy="0 0 0"/>
     <mass value="0.2908090577401484"/>
     <inertia ixx="0.000102" iyy="0.000377" izz="0.000398" ixy="-4.8e-05" iyz="3e-06" ixz="2e-06"/>
@@ -93,5 +93,5 @@
     <origin xyz="0.075 -0.07 0.002768" rpy="0 0 0"/>
     <geometry>
-      <mesh filename="file://$(find IRRobot_description)/meshes/box_motor_4_1.stl" scale="0.001 0.001 0.001"/>
+      <mesh filename="file://$(find irrobot_description)/meshes/box_motor_4_1.stl" scale="0.001 0.001 0.001"/>
     </geometry>
     <material name="silver"/>
@@ -100,5 +100,5 @@
     <origin xyz="0.075 -0.07 0.002768" rpy="0 0 0"/>
     <geometry>
-      <mesh filename="file://$(find IRRobot_description)/meshes/box_motor_4_1.stl" scale="0.001 0.001 0.001"/>
+      <mesh filename="file://$(find irrobot_description)/meshes/box_motor_4_1.stl" scale="0.001 0.001 0.001"/>
     </geometry>
   </collision>
@@ -106,5 +106,5 @@
 <link name="Frente_do_rover_1">
   <inertial>
-    <origin xyz="-0.004484384677440487 -0.05799951148839758 -0.027039271268590424" rpy="0 0 0"/>
+    <origin xyz="-0.004484384677440542 -0.057999511488397326 -0.02703927126859037" rpy="0 0 0"/>
     <mass value="0.5675476589192235"/>
     <inertia ixx="0.002217" iyy="0.000313" izz="0.001971" ixy="0.0" iyz="0.0" ixz="-0.0"/>
@@ -113,5 +113,5 @@
     <origin xyz="0.103 -0.058 -0.063232" rpy="0 0 0"/>
     <geometry>
-      <mesh filename="file://$(find IRRobot_description)/meshes/Frente_do_rover_1.stl" scale="0.001 0.001 0.001"/>
+      <mesh filename="file://$(find irrobot_description)/meshes/Frente_do_rover_1.stl" scale="0.001 0.001 0.001"/>
     </geometry>
     <material name="silver"/>
@@ -120,5 +120,5 @@
     <origin xyz="0.103 -0.058 -0.063232" rpy="0 0 0"/>
     <geometry>
-      <mesh filename="file://$(find IRRobot_description)/meshes/Frente_do_rover_1.stl" scale="0.001 0.001 0.001"/>
+      <mesh filename="file://$(find irrobot_description)/meshes/Frente_do_rover_1.stl" scale="0.001 0.001 0.001"/>
     </geometry>
   </collision>
@@ -126,12 +126,12 @@
 <link name="right_motor_2__1">
   <inertial>
-    <origin xyz="-0.04065000118315213 0.010445876854923236 -2.746126695971074e-07" rpy="0 0 0"/>
+    <origin xyz="-0.040650001183152346 0.01044587685492343 -2.746126695589435e-07" rpy="0 0 0"/>
     <mass value="0.021664868233568425"/>
-    <inertia ixx="1e-06" iyy="1e-06" izz="1e-06" ixy="-0.0" iyz="0.0" ixz="-0.0"/>
+    <inertia ixx="1e-06" iyy="1e-06" izz="1e-06" ixy="0.0" iyz="0.0" ixz="-0.0"/>
   </inertial>
   <visual>
     <origin xyz="-0.0894 0.0915 0.021218" rpy="0 0 0"/>
     <geometry>
-      <mesh filename="file://$(find IRRobot_description)/meshes/right_motor_2__1.stl" scale="0.001 0.001 0.001"/>
+      <mesh filename="file://$(find irrobot_description)/meshes/right_motor_2__1.stl" scale="0.001 0.001 0.001"/>
     </geometry>
     <material name="silver"/>
@@ -140,5 +140,5 @@
     <origin xyz="-0.0894 0.0915 0.021218" rpy="0 0 0"/>
     <geometry>
-      <mesh filename="file://$(find IRRobot_description)/meshes/right_motor_2__1.stl" scale="0.001 0.001 0.001"/>
+      <mesh filename="file://$(find irrobot_description)/meshes/right_motor_2__1.stl" scale="0.001 0.001 0.001"/>
     </geometry>
   </collision>
@@ -146,132 +146,132 @@
 <link name="right_wheel_2_1">
   <inertial>
-    <origin xyz="-0.0011999996572731736 -0.033097991424556564 0.10649972538733041" rpy="0 0 0"/>
+    <origin xyz="-0.0011999996572732152 -0.033097991424556605 0.10649972538733045" rpy="0 0 0"/>
+    <mass value="0.2627861963198363"/>
+    <inertia ixx="8.7e-05" iyy="0.000159" izz="8.7e-05" ixy="0.0" iyz="0.0" ixz="-0.0"/>
+  </inertial>
+  <visual>
+    <origin xyz="-0.0906 0.070282 0.127718" rpy="0 0 0"/>
+    <geometry>
+      <mesh filename="file://$(find irrobot_description)/meshes/right_wheel_2_1.stl" scale="0.001 0.001 0.001"/>
+    </geometry>
+    <material name="silver"/>
+  </visual>
+  <collision>
+    <origin xyz="-0.0906 0.070282 0.127718" rpy="0 0 0"/>
+    <geometry>
+      <mesh filename="file://$(find irrobot_description)/meshes/right_wheel_2_1.stl" scale="0.001 0.001 0.001"/>
+    </geometry>
+  </collision>
+</link>
+<link name="left_motor_2_1">
+  <inertial>
+    <origin xyz="-0.04065000118315238 -0.010445876854922972 -2.746126695762907e-07" rpy="0 0 0"/>
+    <mass value="0.021664868233568425"/>
+    <inertia ixx="1e-06" iyy="1e-06" izz="1e-06" ixy="0.0" iyz="0.0" ixz="0.0"/>
+  </inertial>
+  <visual>
+    <origin xyz="-0.0894 -0.0915 0.021218" rpy="0 0 0"/>
+    <geometry>
+      <mesh filename="file://$(find irrobot_description)/meshes/left_motor_2_1.stl" scale="0.001 0.001 0.001"/>
+    </geometry>
+    <material name="silver"/>
+  </visual>
+  <collision>
+    <origin xyz="-0.0894 -0.0915 0.021218" rpy="0 0 0"/>
+    <geometry>
+      <mesh filename="file://$(find irrobot_description)/meshes/left_motor_2_1.stl" scale="0.001 0.001 0.001"/>
+    </geometry>
+  </collision>
+</link>
+<link name="left_motor_1_1">
+  <inertial>
+    <origin xyz="0.0406500011831524 -0.01044587685492318 -2.74612669493024e-07" rpy="0 0 0"/>
+    <mass value="0.021664868233568425"/>
+    <inertia ixx="1e-06" iyy="1e-06" izz="1e-06" ixy="0.0" iyz="0.0" ixz="0.0"/>
+  </inertial>
+  <visual>
+    <origin xyz="0.0794 -0.0915 0.021218" rpy="0 0 0"/>
+    <geometry>
+      <mesh filename="file://$(find irrobot_description)/meshes/left_motor_1_1.stl" scale="0.001 0.001 0.001"/>
+    </geometry>
+    <material name="silver"/>
+  </visual>
+  <collision>
+    <origin xyz="0.0794 -0.0915 0.021218" rpy="0 0 0"/>
+    <geometry>
+      <mesh filename="file://$(find irrobot_description)/meshes/left_motor_1_1.stl" scale="0.001 0.001 0.001"/>
+    </geometry>
+  </collision>
+</link>
+<link name="right_motor_1_1">
+  <inertial>
+    <origin xyz="0.040650001183152686 0.01044587685492275 -2.7461266954159624e-07" rpy="0 0 0"/>
+    <mass value="0.021664868233568425"/>
+    <inertia ixx="1e-06" iyy="1e-06" izz="1e-06" ixy="0.0" iyz="0.0" ixz="-0.0"/>
+  </inertial>
+  <visual>
+    <origin xyz="0.0794 0.0915 0.021218" rpy="0 0 0"/>
+    <geometry>
+      <mesh filename="file://$(find irrobot_description)/meshes/right_motor_1_1.stl" scale="0.001 0.001 0.001"/>
+    </geometry>
+    <material name="silver"/>
+  </visual>
+  <collision>
+    <origin xyz="0.0794 0.0915 0.021218" rpy="0 0 0"/>
+    <geometry>
+      <mesh filename="file://$(find irrobot_description)/meshes/right_motor_1_1.stl" scale="0.001 0.001 0.001"/>
+    </geometry>
+  </collision>
+</link>
+<link name="left_wheel_1_1">
+  <inertial>
+    <origin xyz="0.2021999996572732 0.033097991424556494 -0.06230027461266955" rpy="0 0 0"/>
+    <mass value="0.2627861963198363"/>
+    <inertia ixx="8.7e-05" iyy="0.000159" izz="8.7e-05" ixy="-0.0" iyz="0.0" ixz="0.0"/>
+  </inertial>
+  <visual>
+    <origin xyz="0.2816 -0.070282 -0.041082" rpy="0 0 0"/>
+    <geometry>
+      <mesh filename="file://$(find irrobot_description)/meshes/left_wheel_1_1.stl" scale="0.001 0.001 0.001"/>
+    </geometry>
+    <material name="silver"/>
+  </visual>
+  <collision>
+    <origin xyz="0.2816 -0.070282 -0.041082" rpy="0 0 0"/>
+    <geometry>
+      <mesh filename="file://$(find irrobot_description)/meshes/left_wheel_1_1.stl" scale="0.001 0.001 0.001"/>
+    </geometry>
+  </collision>
+</link>
+<link name="left_wheel_2_1">
+  <inertial>
+    <origin xyz="-0.20219999965727337 0.03309799142455655 -0.10650027461266962" rpy="0 0 0"/>
+    <mass value="0.2627861963198363"/>
+    <inertia ixx="8.7e-05" iyy="0.000159" izz="8.7e-05" ixy="-0.0" iyz="0.0" ixz="0.0"/>
+  </inertial>
+  <visual>
+    <origin xyz="-0.2916 -0.070282 -0.085282" rpy="0 0 0"/>
+    <geometry>
+      <mesh filename="file://$(find irrobot_description)/meshes/left_wheel_2_1.stl" scale="0.001 0.001 0.001"/>
+    </geometry>
+    <material name="silver"/>
+  </visual>
+  <collision>
+    <origin xyz="-0.2916 -0.070282 -0.085282" rpy="0 0 0"/>
+    <geometry>
+      <mesh filename="file://$(find irrobot_description)/meshes/left_wheel_2_1.stl" scale="0.001 0.001 0.001"/>
+    </geometry>
+  </collision>
+</link>
+<link name="right_wheel_1_1">
+  <inertial>
+    <origin xyz="0.001199999657273229 -0.033097991424556744 0.06229972538733042" rpy="0 0 0"/>
     <mass value="0.2627861963198363"/>
     <inertia ixx="8.7e-05" iyy="0.000159" izz="8.7e-05" ixy="0.0" iyz="0.0" ixz="0.0"/>
   </inertial>
   <visual>
-    <origin xyz="-0.0906 0.070282 0.127718" rpy="0 0 0"/>
-    <geometry>
-      <mesh filename="file://$(find IRRobot_description)/meshes/right_wheel_2_1.stl" scale="0.001 0.001 0.001"/>
-    </geometry>
-    <material name="silver"/>
-  </visual>
-  <collision>
-    <origin xyz="-0.0906 0.070282 0.127718" rpy="0 0 0"/>
-    <geometry>
-      <mesh filename="file://$(find IRRobot_description)/meshes/right_wheel_2_1.stl" scale="0.001 0.001 0.001"/>
-    </geometry>
-  </collision>
-</link>
-<link name="left_motor_2_1">
-  <inertial>
-    <origin xyz="-0.040650001183152186 -0.01044587685492318 -2.7461266959363795e-07" rpy="0 0 0"/>
-    <mass value="0.021664868233568425"/>
-    <inertia ixx="1e-06" iyy="1e-06" izz="1e-06" ixy="0.0" iyz="0.0" ixz="0.0"/>
-  </inertial>
-  <visual>
-    <origin xyz="-0.0894 -0.0915 0.021218" rpy="0 0 0"/>
-    <geometry>
-      <mesh filename="file://$(find IRRobot_description)/meshes/left_motor_2_1.stl" scale="0.001 0.001 0.001"/>
-    </geometry>
-    <material name="silver"/>
-  </visual>
-  <collision>
-    <origin xyz="-0.0894 -0.0915 0.021218" rpy="0 0 0"/>
-    <geometry>
-      <mesh filename="file://$(find IRRobot_description)/meshes/left_motor_2_1.stl" scale="0.001 0.001 0.001"/>
-    </geometry>
-  </collision>
-</link>
-<link name="left_motor_1_1">
-  <inertial>
-    <origin xyz="0.04065000118315222 -0.01044587685492293 -2.7461266960751574e-07" rpy="0 0 0"/>
-    <mass value="0.021664868233568425"/>
-    <inertia ixx="1e-06" iyy="1e-06" izz="1e-06" ixy="0.0" iyz="0.0" ixz="0.0"/>
-  </inertial>
-  <visual>
-    <origin xyz="0.0794 -0.0915 0.021218" rpy="0 0 0"/>
-    <geometry>
-      <mesh filename="file://$(find IRRobot_description)/meshes/left_motor_1_1.stl" scale="0.001 0.001 0.001"/>
-    </geometry>
-    <material name="silver"/>
-  </visual>
-  <collision>
-    <origin xyz="0.0794 -0.0915 0.021218" rpy="0 0 0"/>
-    <geometry>
-      <mesh filename="file://$(find IRRobot_description)/meshes/left_motor_1_1.stl" scale="0.001 0.001 0.001"/>
-    </geometry>
-  </collision>
-</link>
-<link name="right_motor_1_1">
-  <inertial>
-    <origin xyz="0.04065000118315217 0.010445876854922917 -2.746126695832296e-07" rpy="0 0 0"/>
-    <mass value="0.021664868233568425"/>
-    <inertia ixx="1e-06" iyy="1e-06" izz="1e-06" ixy="-0.0" iyz="0.0" ixz="-0.0"/>
-  </inertial>
-  <visual>
-    <origin xyz="0.0794 0.0915 0.021218" rpy="0 0 0"/>
-    <geometry>
-      <mesh filename="file://$(find IRRobot_description)/meshes/right_motor_1_1.stl" scale="0.001 0.001 0.001"/>
-    </geometry>
-    <material name="silver"/>
-  </visual>
-  <collision>
-    <origin xyz="0.0794 0.0915 0.021218" rpy="0 0 0"/>
-    <geometry>
-      <mesh filename="file://$(find IRRobot_description)/meshes/right_motor_1_1.stl" scale="0.001 0.001 0.001"/>
-    </geometry>
-  </collision>
-</link>
-<link name="left_wheel_1_1">
-  <inertial>
-    <origin xyz="0.20219999965727312 0.033097991424556605 -0.06230027461266961" rpy="0 0 0"/>
-    <mass value="0.2627861963198363"/>
-    <inertia ixx="8.7e-05" iyy="0.000159" izz="8.7e-05" ixy="-0.0" iyz="0.0" ixz="-0.0"/>
-  </inertial>
-  <visual>
-    <origin xyz="0.2816 -0.070282 -0.041082" rpy="0 0 0"/>
-    <geometry>
-      <mesh filename="file://$(find IRRobot_description)/meshes/left_wheel_1_1.stl" scale="0.001 0.001 0.001"/>
-    </geometry>
-    <material name="silver"/>
-  </visual>
-  <collision>
-    <origin xyz="0.2816 -0.070282 -0.041082" rpy="0 0 0"/>
-    <geometry>
-      <mesh filename="file://$(find IRRobot_description)/meshes/left_wheel_1_1.stl" scale="0.001 0.001 0.001"/>
-    </geometry>
-  </collision>
-</link>
-<link name="left_wheel_2_1">
-  <inertial>
-    <origin xyz="-0.20219999965727342 0.03309799142455665 -0.10650027461266964" rpy="0 0 0"/>
-    <mass value="0.2627861963198363"/>
-    <inertia ixx="8.7e-05" iyy="0.000159" izz="8.7e-05" ixy="-0.0" iyz="-0.0" ixz="0.0"/>
-  </inertial>
-  <visual>
-    <origin xyz="-0.2916 -0.070282 -0.085282" rpy="0 0 0"/>
-    <geometry>
-      <mesh filename="file://$(find IRRobot_description)/meshes/left_wheel_2_1.stl" scale="0.001 0.001 0.001"/>
-    </geometry>
-    <material name="silver"/>
-  </visual>
-  <collision>
-    <origin xyz="-0.2916 -0.070282 -0.085282" rpy="0 0 0"/>
-    <geometry>
-      <mesh filename="file://$(find IRRobot_description)/meshes/left_wheel_2_1.stl" scale="0.001 0.001 0.001"/>
-    </geometry>
-  </collision>
-</link>
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
File: urdf/IRRobot_description/urdf/materials.xacro (robot description, xacro)
@@ -1,4 +1,4 @@
 <?xml version="1.0" ?>
-<robot name="IRRobot" xmlns:xacro="http://www.ros.org/wiki/xacro" >
+<robot name="irrobot" xmlns:xacro="http://www.ros.org/wiki/xacro" >
 <material name="silver">
   <color rgba="0.700 0.700 0.700 1.000"/>
